File: breakout-v2.brd (EAGLE design)
At the start: 32.7 x 34.3 mm, 3 parts

Commit message: breakout board v2
Parts:
- moved RIGHT 74.3 mm to (-35.6, 35.6), turned to 0 degrees
- moved U$1 45.4 mm to (-27.9, 1.27)
- moved LEFT 44.5 mm to (-35.6, 30.5), turned to 0 degrees
Routing:
- net GPIO3: track 19.3 -> 0.00 mm
- net GPIO2: track 18.0 -> 0.00 mm
- net GPIO4: track 17.3 -> 0.00 mm
- net GPIO1: track 16.3 -> 0.00 mm
- net GPIO5: track 13.6 -> 0.00 mm
- net GPIO0: track 13.2 -> 0.00 mm
- net GPIO6: track 11.9 -> 0.00 mm
- net SPICSN: track 7.65 -> 0.00 mm
- net SPICLK: track 7.42 -> 0.00 mm
- net EXTON: track 7.29 -> 0.00 mm
- net GPIO8: track 7.14 -> 0.00 mm
- net VSS: track 7.00 -> 0.00 mm
- net SPIMOSI: track 6.97 -> 0.00 mm
- net SPIMISO: track 6.84 -> 0.00 mm
- net WAKEUP: track 6.80 -> 0.00 mm
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- removed copper zone on layer 1, net VSS
Other:
- board size 32.7 x 34.3 mm -> 100 x 80 mm
